Commit message: proper urdf pushed

File: Robotic_arm_urdf_v2/urdf/Robotic_arm_urdf_v2.urdf (robot description, URDF)
Before this commit: robot Robotic_arm_urdf, 7 links, 6 joints
Links:
- removed link arm1_link
- removed link arm2_link
- removed link bicep_link
- removed link gripperSup_link
- removed link leftClaw_link
- removed link rightClaw_link
- added link arm1_Link, mass 0.0713721391109546; collision mesh filename=package://Robotic_arm_urdf_v2/meshes/arm1_Link.STL; visual mesh filename=package://Robotic_arm_urdf_v2/meshes/arm1_Link.STL
- added link arm2_Link, mass 0.059726655007088; collision mesh filename=package://Robotic_arm_urdf_v2/meshes/arm2_Link.STL; visual mesh filename=package://Robotic_arm_urdf_v2/meshes/arm2_Link.STL
- added link bicep_Link, mass 0.176834526977706; collision mesh filename=package://Robotic_arm_urdf_v2/meshes/bicep_Link.STL; visual mesh filename=package://Robotic_arm_urdf_v2/meshes/bicep_Link.STL
- added link gripperSup_Link, mass 0.0107802680605055; collision mesh filename=package://Robotic_arm_urdf_v2/meshes/gripperSup_Link.STL; visual mesh filename=package://Robotic_arm_urdf_v2/meshes/gripperSup_Link.STL
- added link leftClaw_Link, mass 0.00659380087326398; collision mesh filename=package://Robotic_arm_urdf_v2/meshes/leftClaw_Link.STL; visual mesh filename=package://Robotic_arm_urdf_v2/meshes/leftClaw_Link.STL
- added link rightClaw_Link, mass 0.00659380087326398; collision mesh filename=package://Robotic_arm_urdf_v2/meshes/rightClaw_Link.STL; visual mesh filename=package://Robotic_arm_urdf_v2/meshes/rightClaw_Link.STL
- link base_link: geometry collision mesh filename=package://Robotic_arm_urdf_v2/meshes/base_link.STL; visual mesh filename=package://Robotic_arm_urdf_v2/meshes/base_link.STL
Joints:
- joint arm1_joint: child arm1_link -> arm1_Link; limit lower=-1 upper=1.5708 effort=5 velocity=1 -> lower=0 upper=0 effort=0 velocity=0; origin xyz=0.040988 -0.049174 0.050067 rpy=1.5708 0 -0.64651 -> xyz=0.049445 -0.037317 0.056597 rpy=1.5708 0 -0.64651; parent bicep_link -> bicep_Link
- joint arm2_joint: child arm2_link -> arm2_Link; limit lower=0 upper=1.5708 effort=5 velocity=1 -> lower=0 upper=0 effort=0 velocity=0; origin xyz=-0.0028592 0.13609 -0.025068 rpy=-3.1416 0 0 -> xyz=-0.0078188 0.12976 0 rpy=-3.1416 0 0; parent arm1_link -> arm1_Link
- joint bicep_joint: child bicep_link -> bicep_Link; limit lower=-12.5664 upper=12.5664 effort=5 velocity=1 -> lower=0 upper=0 effort=0 velocity=0; origin xyz=-0.04099 -0.17922 0.1611 rpy=0 0 0 -> xyz=0 0 0.0655 rpy=0 0 0
- joint gripperSup_joint: child gripperSup_link -> gripperSup_Link; origin xyz=-0.14874 -0.0058338 0.0019915 rpy=1.5708 -0.64688 0.039202 -> xyz=-0.14338 -0.0056238 0.0125 rpy=1.5708 -0.64688 0.039202; parent arm2_link -> arm2_Link
- joint leftClaw_joint: child leftClaw_link -> leftClaw_Link; limit lower=-1.5708 upper=0 effort=5 velocity=1 -> lower=0 upper=0 effort=0 velocity=0; parent gripperSup_link -> gripperSup_Link
- joint rightClaw_joint: child rightClaw_link -> rightClaw_Link; limit lower=0 upper=1.5708 effort=5 velocity=1 -> lower=0 upper=0 effort=0 velocity=0; parent gripperSup_link -> gripperSup_Link

File: robotic_arm_ws/src/robotic_arm/urdf/Robotic_arm_urdf_v2.urdf (robot description, URDF)
Before this commit: robot Robotic_arm_urdf, 7 links, 6 joints
Links:
- removed link arm1_link
- removed link arm2_link
- removed link bicep_link
- removed link gripperSup_link
- removed link leftClaw_link
- removed link rightClaw_link
- added link arm1_Link, mass 0.0713721391109546; collision mesh filename=package://Robotic_arm_urdf_v2/meshes/arm1_Link.STL; visual mesh filename=package://Robotic_arm_urdf_v2/meshes/arm1_Link.STL
- added link arm2_Link, mass 0.059726655007088; collision mesh filename=package://Robotic_arm_urdf_v2/meshes/arm2_Link.STL; visual mesh filename=package://Robotic_arm_urdf_v2/meshes/arm2_Link.STL
- added link bicep_Link, mass 0.176834526977706; collision mesh filename=package://Robotic_arm_urdf_v2/meshes/bicep_Link.STL; visual mesh filename=package://Robotic_arm_urdf_v2/meshes/bicep_Link.STL
- added link gripperSup_Link, mass 0.0107802680605055; collision mesh filename=package://Robotic_arm_urdf_v2/meshes/gripperSup_Link.STL; visual mesh filename=package://Robotic_arm_urdf_v2/meshes/gripperSup_Link.STL
- added link leftClaw_Link, mass 0.00659380087326398; collision mesh filename=package://Robotic_arm_urdf_v2/meshes/leftClaw_Link.STL; visual mesh filename=package://Robotic_arm_urdf_v2/meshes/leftClaw_Link.STL
- added link rightClaw_Link, mass 0.00659380087326398; collision mesh filename=package://Robotic_arm_urdf_v2/meshes/rightClaw_Link.STL; visual mesh filename=package://Robotic_arm_urdf_v2/meshes/rightClaw_Link.STL
- link base_link: geometry collision mesh filename=package://Robotic_arm_urdf_v2/meshes/base_link.STL; visual mesh filename=package://Robotic_arm_urdf_v2/meshes/base_link.STL
Joints:
- joint arm1_joint: child arm1_link -> arm1_Link; origin xyz=0.040988 -0.049174 0.050067 rpy=1.5708 0 -0.64651 -> xyz=0.049445 -0.037317 0.056597 rpy=1.5708 0 -0.64651; parent bicep_link -> bicep_Link
- joint arm2_joint: child arm2_link -> arm2_Link; origin xyz=-0.0028592 0.13609 -0.025068 rpy=-3.1416 0 0 -> xyz=-0.0078188 0.12976 0 rpy=-3.1416 0 0; parent arm1_link -> arm1_Link
- joint bicep_joint: child bicep_link -> bicep_Link; origin xyz=-0.04099 -0.17922 0.1611 rpy=0 0 0 -> xyz=0 0 0.0655 rpy=0 0 0
- joint gripperSup_joint: child gripperSup_link -> gripperSup_Link; origin xyz=-0.14874 -0.0058338 0.0019915 rpy=1.5708 -0.64688 0.039202 -> xyz=-0.14338 -0.0056238 0.0125 rpy=1.5708 -0.64688 0.039202; parent arm2_link -> arm2_Link
- joint leftClaw_joint: child leftClaw_link -> leftClaw_Link; parent gripperSup_link -> gripperSup_Link
- joint rightClaw_joint: child rightClaw_link -> rightClaw_Link; parent gripperSup_link -> gripperSup_Link
