Commit message: Right claw changed in urdf

File: Robotic_arm_urdf/urdf/Robotic_arm_urdf.urdf (robot description, URDF)
Before this commit: robot Robotic_arm_urdf_v2, 7 links, 6 joints
Links:
- removed link base_link
- added link base_Link, mass 0.273457775165078; collision mesh filename=package://Robotic_arm_urdf/meshes/base_Link.STL; visual mesh filename=package://Robotic_arm_urdf/meshes/base_Link.STL
- link arm1_Link: mass 0.0713721391109546 -> 0.0713721391109545; geometry collision mesh filename=package://Robotic_arm_urdf/meshes/arm1_Link.STL; visual mesh filename=package://Robotic_arm_urdf/meshes/arm1_Link.STL
- link arm2_Link: geometry collision mesh filename=package://Robotic_arm_urdf/meshes/arm2_Link.STL; visual mesh filename=package://Robotic_arm_urdf/meshes/arm2_Link.STL
- link bicep_Link: geometry collision mesh filename=package://Robotic_arm_urdf/meshes/bicep_Link.STL; visual mesh filename=package://Robotic_arm_urdf/meshes/bicep_Link.STL
- link gripperSup_Link: geometry collision mesh filename=package://Robotic_arm_urdf/meshes/gripperSup_Link.STL; visual mesh filename=package://Robotic_arm_urdf/meshes/gripperSup_Link.STL
- link leftClaw_Link: geometry collision mesh filename=package://Robotic_arm_urdf/meshes/leftClaw_Link.STL; visual mesh filename=package://Robotic_arm_urdf/meshes/leftClaw_Link.STL
- link rightClaw_Link: mass 0.00659380087326398 -> 0.00702806279088024; geometry collision mesh filename=package://Robotic_arm_urdf/meshes/rightClaw_Link.STL; visual mesh filename=package://Robotic_arm_urdf/meshes/rightClaw_Link.STL
Joints:
- joint arm1_joint: origin xyz=0.049445 -0.037317 0.056597 rpy=1.5708 0 -0.64651 -> xyz=0.0494451953137995 -0.0373170501614636 0.0565970142948164 rpy=1.5707963267949 0 -0.646512137978303
- joint arm2_joint: origin xyz=-0.0078188 0.12976 0 rpy=-3.1416 0 0 -> xyz=-0.00781878999246252 0.129764658220391 0 rpy=-3.14159265358979 0 0
- joint bicep_joint: origin xyz=0 0 0.0655 rpy=0 0 0 -> xyz=0 0 0.0655000000000001 rpy=0 0 0; parent base_link -> base_Link
- joint gripperSup_joint: origin xyz=-0.14338 -0.0056238 0.0125 rpy=1.5708 -0.64688 0.039202 -> xyz=-0.14338485066181 -0.00562384447952546 0.0125 rpy=1.5707963267949 -0.646881742667799 0.0392019328832376
- joint leftClaw_joint: origin xyz=-0.03814 0.011889 0.003 rpy=0 0 0 -> xyz=-0.0381397989509513 0.0118888339315903 0.00300000000000006 rpy=0 0 0
- joint rightClaw_joint: origin xyz=-0.021867 0.033434 0.003 rpy=0 0 0 -> xyz=-0.0218668699706155 0.0334339443374561 0.003 rpy=0 0 0

File: robotic_arm_ws/src/robotic_arm/urdf/Robotic_arm_urdf.urdf (robot description, URDF)
Before this commit: robot Robotic_arm_urdf_v2, 7 links, 6 joints
Links:
- link arm1_Link: mass 0.0713721391109546 -> 0.0713721391109545; geometry collision mesh filename=package://Robotic_arm_urdf/meshes/arm1_Link.STL; visual mesh filename=package://Robotic_arm_urdf/meshes/arm1_Link.STL
- link arm2_Link: geometry collision mesh filename=package://Robotic_arm_urdf/meshes/arm2_Link.STL; visual mesh filename=package://Robotic_arm_urdf/meshes/arm2_Link.STL
- link base_Link: geometry collision mesh filename=package://Robotic_arm_urdf/meshes/base_Link.STL; visual mesh filename=package://Robotic_arm_urdf/meshes/base_Link.STL
- link bicep_Link: geometry collision mesh filename=package://Robotic_arm_urdf/meshes/bicep_Link.STL; visual mesh filename=package://Robotic_arm_urdf/meshes/bicep_Link.STL
- link gripperSup_Link: geometry collision mesh filename=package://Robotic_arm_urdf/meshes/gripperSup_Link.STL; visual mesh filename=package://Robotic_arm_urdf/meshes/gripperSup_Link.STL
- link leftClaw_Link: geometry collision mesh filename=package://Robotic_arm_urdf/meshes/leftClaw_Link.STL; visual mesh filename=package://Robotic_arm_urdf/meshes/leftClaw_Link.STL
- link rightClaw_Link: mass 0.00659380087326398 -> 0.00702806279088024; geometry collision mesh filename=package://Robotic_arm_urdf/meshes/rightClaw_Link.STL; visual mesh filename=package://Robotic_arm_urdf/meshes/rightClaw_Link.STL
Joints:
- joint arm1_joint: limit lower=-1.5707963267949 upper=1.000000000000001 effort=7.0 velocity=0.7 -> lower=0 upper=0 effort=0 velocity=0; origin xyz=0.049445 -0.037317 0.056597 rpy=1.5708 0 -0.64651 -> xyz=0.0494451953137995 -0.0373170501614636 0.0565970142948164 rpy=1.5707963267949 0 -0.646512137978303
- joint arm2_joint: limit lower=-1.5707963267949 upper=1.000000000000001 effort=7.0 velocity=0.7 -> lower=0 upper=0 effort=0 velocity=0; origin xyz=-0.0078188 0.12976 0 rpy=-3.1416 0 0 -> xyz=-0.00781878999246252 0.129764658220391 0 rpy=-3.14159265358979 0 0
- joint bicep_joint: limit lower=-6.28318530717959 upper=6.28318530717959 effort=7.0 velocity=0.7 -> lower=0 upper=0 effort=0 velocity=0; origin xyz=0 0 0.0655 rpy=0 0 0 -> xyz=0 0 0.0655000000000001 rpy=0 0 0
- joint gripperSup_joint: origin xyz=-0.14338 -0.0056238 0.0125 rpy=1.5708 -0.64688 0.039202 -> xyz=-0.14338485066181 -0.00562384447952546 0.0125 rpy=1.5707963267949 -0.646881742667799 0.0392019328832376
- joint leftClaw_joint: limit lower=-1.5707963267949 upper=0 effort=7.0 velocity=0.7 -> lower=0 upper=0 effort=0 velocity=0; origin xyz=-0.03814 0.011889 0.003 rpy=0 0 0 -> xyz=-0.0381397989509513 0.0118888339315903 0.00300000000000006 rpy=0 0 0
- joint rightClaw_joint: limit lower=0 upper=1.5707963267949 effort=7.0 velocity=0.7 -> lower=0 upper=0 effort=0 velocity=0; origin xyz=-0.021867 0.033434 0.003 rpy=0 0 0 -> xyz=-0.0218668699706155 0.0334339443374561 0.003 rpy=0 0 0
