Commit message: Right Claw needs to be changed

File: robotic_arm_ws/src/robotic_arm/urdf/Robotic_arm_urdf.urdf (robot description, URDF)
Before this commit: robot Robotic_arm_urdf_v2, 7 links, 6 joints
Links:
- removed link base_link
- added link base_Link, mass 0.273457775165078; collision mesh filename=package://robotic_arm/meshes/base_Link.STL; visual mesh filename=package://robotic_arm/meshes/base_Link.STL
- link arm1_Link: geometry collision mesh filename=package://robotic_arm/meshes/arm1_Link.STL; visual mesh filename=package://robotic_arm/meshes/arm1_Link.STL
- link arm2_Link: geometry collision mesh filename=package://robotic_arm/meshes/arm2_Link.STL; visual mesh filename=package://robotic_arm/meshes/arm2_Link.STL
- link bicep_Link: geometry collision mesh filename=package://robotic_arm/meshes/bicep_Link.STL; visual mesh filename=package://robotic_arm/meshes/bicep_Link.STL
- link gripperSup_Link: geometry collision mesh filename=package://robotic_arm/meshes/gripperSup_Link.STL; visual mesh filename=package://robotic_arm/meshes/gripperSup_Link.STL
- link leftClaw_Link: geometry collision mesh filename=package://robotic_arm/meshes/leftClaw_Link.STL; visual mesh filename=package://robotic_arm/meshes/leftClaw_Link.STL
- link rightClaw_Link: geometry collision mesh filename=package://robotic_arm/meshes/rightClaw_Link.STL; visual mesh filename=package://robotic_arm/meshes/rightClaw_Link.STL
Joints:
- joint arm1_joint: limit lower=0 upper=0 effort=0 velocity=0 -> lower=-1.5707963267949 upper=1.000000000000001 effort=7.0 velocity=0.7
- joint arm2_joint: limit lower=0 upper=0 effort=0 velocity=0 -> lower=-1.5707963267949 upper=1.000000000000001 effort=7.0 velocity=0.7
- joint bicep_joint: limit lower=0 upper=0 effort=0 velocity=0 -> lower=-6.28318530717959 upper=6.28318530717959 effort=7.0 velocity=0.7; parent base_link -> base_Link
- joint leftClaw_joint: limit lower=0 upper=0 effort=0 velocity=0 -> lower=-1.5707963267949 upper=0 effort=7.0 velocity=0.7
- joint rightClaw_joint: limit lower=0 upper=0 effort=0 velocity=0 -> lower=0 upper=1.5707963267949 effort=7.0 velocity=0.7

Commit message: urdf

File: robotic_arm_ws/src/robotic_arm/urdf/Robotic_arm_urdf.urdf (robot description, URDF)
Before this commit: robot Robotic_arm_urdf, 7 links, 6 joints
Links:
- link arm1_Link: geometry collision mesh filename=package://robotic_arm/meshes/arm1_Link.STL; visual mesh filename=package://robotic_arm/meshes/arm1_Link.STL
- link arm2_Link: geometry collision mesh filename=package://robotic_arm/meshes/arm2_Link.STL; visual mesh filename=package://robotic_arm/meshes/arm2_Link.STL
- link base_Link: geometry collision mesh filename=package://robotic_arm/meshes/base_Link.STL; visual mesh filename=package://robotic_arm/meshes/base_Link.STL
- link bicep_Link: geometry collision mesh filename=package://robotic_arm/meshes/bicep_Link.STL; visual mesh filename=package://robotic_arm/meshes/bicep_Link.STL
- link gripperSup_Link: geometry collision mesh filename=package://robotic_arm/meshes/gripperSup_Link.STL; visual mesh filename=package://robotic_arm/meshes/gripperSup_Link.STL
- link leftClaw_Link: geometry collision mesh filename=package://robotic_arm/meshes/leftClaw_Link.STL; visual mesh filename=package://robotic_arm/meshes/leftClaw_Link.STL
- link rightClaw_Link: geometry collision mesh filename=package://robotic_arm/meshes/rightClaw_Link.STL; visual mesh filename=package://robotic_arm/meshes/rightClaw_Link.STL
Joints:
- joint arm1_joint: limit lower=0 upper=0 effort=0 velocity=0 -> lower=-0.975325981771001 upper=1.000000000000001 effort=7.0 velocity=0.7
- joint arm2_joint: limit lower=0 upper=0 effort=0 velocity=0 -> lower=0 upper=1.000000000000001 effort=7.0 velocity=0.7
- joint bicep_joint: limit lower=0 upper=0 effort=0 velocity=0 -> lower=-6.28318530717959 upper=6.28318530717959 effort=7.0 velocity=0.7
- joint leftClaw_joint: limit lower=0 upper=0 effort=0 velocity=0 -> lower=-1.5707963267949 upper=0 effort=7.0 velocity=0.7
- joint rightClaw_joint: limit lower=0 upper=0 effort=0 velocity=0 -> lower=0 upper=1.5707963267949 effort=7.0 velocity=0.7
