Commit message: changed package name to robotic_arm_description

File: robotic_arm_ws/src/robotic_arm_description/urdf/Robotic_arm_urdf.urdf (robot description, URDF)
Before this commit: robot Robotic_arm_urdf, 7 links, 6 joints
Links:
- link arm1_Link: geometry collision mesh filename=package://robotic_arm_description/meshes/arm1_Link.STL; visual mesh filename=package://robotic_arm_description/meshes/arm1_Link.STL
- link arm2_Link: geometry collision mesh filename=package://robotic_arm_description/meshes/arm2_Link.STL; visual mesh filename=package://robotic_arm_description/meshes/arm2_Link.STL
- link base_Link: geometry collision mesh filename=package://robotic_arm_description/meshes/base_Link.STL; visual mesh filename=package://robotic_arm_description/meshes/base_Link.STL
- link bicep_Link: geometry collision mesh filename=package://robotic_arm_description/meshes/bicep_Link.STL; visual mesh filename=package://robotic_arm_description/meshes/bicep_Link.STL
- link gripperSup_Link: geometry collision mesh filename=package://robotic_arm_description/meshes/gripperSup_Link.STL; visual mesh filename=package://robotic_arm_description/meshes/gripperSup_Link.STL
- link leftClaw_Link: geometry collision mesh filename=package://robotic_arm_description/meshes/leftClaw_Link.STL; visual mesh filename=package://robotic_arm_description/meshes/leftClaw_Link.STL
- link rightClaw_Link: geometry collision mesh filename=package://robotic_arm_description/meshes/rightClaw_Link.STL; visual mesh filename=package://robotic_arm_description/meshes/rightClaw_Link.STL
Joints:
- joint arm1_joint: limit lower=-0.975325981771001 upper=1.000000000000001 effort=7.0 velocity=0.7 -> lower=-0.975325981771001 upper=1.000000000000001 effort=30 velocity=10
- joint arm2_joint: limit lower=0 upper=1.000000000000001 effort=7.0 velocity=0.7 -> lower=0 upper=1.000000000000001 effort=30 velocity=10
- joint bicep_joint: limit lower=-6.28318530717959 upper=6.28318530717959 effort=7.0 velocity=0.7 -> lower=-6.28318530717959 upper=6.28318530717959 effort=30.0 velocity=10
- joint leftClaw_joint: limit lower=-1.5707963267949 upper=0 effort=7.0 velocity=0.7 -> lower=-1.5707963267949 upper=0 effort=30 velocity=10
- joint rightClaw_joint: limit lower=0 upper=1.5707963267949 effort=7.0 velocity=0.7 -> lower=0 upper=1.5707963267949 effort=30 velocity=10; mimic (none) -> joint=leftClaw_joint multiplier=-1

Commit message: urdf and launch file modifications

File: robotic_arm_ws/src/robotic_arm_description/urdf/Robotic_arm_urdf.urdf (robot description, URDF)
Before this commit: robot Robotic_arm_urdf, 7 links, 6 joints
Joints:
- joint arm2_joint: limit lower=0 upper=1.000000000000001 effort=30 velocity=10 -> lower=0 upper=1.5707963267949 effort=30 velocity=10
