Commit message: ros2 control hardiware interface configuration file + gazebo ros2 control tag

File: robotic_arm_ws/src/robotic_arm_description/urdf/robotic_arm.urdf.xacro (robot description, xacro)
@@ -1,8 +1,8 @@
 <?xml version="1.0"?>
-<!-- This URDF was automatically created by SolidWorks to URDF Exporter!
-     Originally created by Stephen Brawner (brawner@gmail.com)
-     Commit Version: 1.6.0-4-g7f85cfe  Build Version: 1.6.7995.38578
-     For more information, please see http://wiki.ros.org/sw_urdf_exporter -->
-<robot xmlns:xacro="http://www.ros.org/wiki/xacro" name="Robotic_arm_urdf">
+<robot xmlns:xacro="http://www.ros.org/wiki/xacro" name="robotic_arm_urdf">
+  <!-- Include Gazebo parameters -->
+  <xacro:include filename="$(find robotic_arm_description)/urdf/robotic_arm_gazebo.xacro"/>
+  <xacro:include filename="$(find robotic_arm_description)/urdf/robotic_arm_ros2_control.xacro"/>
+  <xacro:property name="PI" value="3.14159265359"/>
   <!-- =========================
        BASE LINK
@@ -62,5 +62,5 @@
     <child link="bicep_Link"/>
     <axis xyz="0 0 1"/>
-    <limit lower="-6.28318530717959" upper="6.28318530717959" effort="30.0" velocity="10"/>
+    <limit lower="${-PI}" upper="${PI}" effort="30.0" velocity="10"/>
   </joint>
   <!-- =========================
@@ -96,5 +96,5 @@
     <child link="arm1_Link"/>
     <axis xyz="0 0 -1"/>
-    <limit lower="-0.975325981771001" upper="1.000000000000001" effort="30" velocity="10"/>
+    <limit lower="${-PI / 2}" upper="${PI / 2}" effort="30" velocity="10"/>
   </joint>
   <!-- =========================
@@ -231,11 +231,3 @@
     <mimic joint="leftClaw_joint" multiplier="-1"/>
   </joint>
-  <!-- =========================
-       GAZEBO GAZEBO PLUGIN
-  ============================ -->
-  <!-- <gazebo>
-    <plugin filename="gz_ros2_control-system" name="gz_ros2_control::GazeboSimROS2ControlPlugin">
-        <parameters></parameters>
-    </plugin>
-  </gazebo> -->
 </robot>

Commit message: Physical robot urdf configuration and launch  file are finished

File: robotic_arm_ws/src/robotic_arm_description/urdf/robotic_arm.urdf.xacro (robot description, xacro)
@@ -1,4 +1,5 @@
 <?xml version="1.0"?>
 <robot xmlns:xacro="http://www.ros.org/wiki/xacro" name="robotic_arm_urdf">
+  <xacro:arg name="is_sim" default="true"/>
   <!-- Include Gazebo parameters -->
   <xacro:include filename="$(find robotic_arm_description)/urdf/robotic_arm_gazebo.xacro"/>

File: robotic_arm_ws/src/robotic_arm_description/urdf/robotic_arm_ros2_control.xacro (robot description, xacro)
@@ -1,13 +1,24 @@
 <?xml version="1.0"?>
 <robot xmlns:xacro="http://www.ros.org/wiki/xacro" name="robotic_arm_urdf">
-  <xacro:property name="PI" value="3.14159265359"/>
     <!-- Ros2 control plugin  -->
     <ros2_control type="system" name="RobotSystem">
-         <hardware>
-            <plugin>gz_ros2_control/GazeboSimSystem</plugin>
-         </hardware>
-         <!-- <hardware>
-            Here will be another hardware tag for the real robot
-         </hardware> -->
+        <xacro:property name="PI" value="3.14159265359"/>
+        <!-- ros2_control gazebo -->
+         <xacro:if value="$(arg is_sim)">
+            <hardware>
+                <plugin>gz_ros2_control/GazeboSimSystem</plugin> <!--  Gazebo harware interface  -->
+            </hardware>
+            <joint name="rightClaw_joint">
+                <param name="mimic">leftClaw_joint</param>
+                <param name="multiplier">-1</param>
+            </joint>
+         </xacro:if>
+         <!-- ros2_control real robot -->
+         <xacro:unless value="$(arg is_sim)">
+            <hardware>
+                <plugin>robotic_arm_controllers/RoboticArmInterface</plugin>
+                <param name="port">/dev/ttyUSB0</param>
+            </hardware>
+         </xacro:unless>
         <joint name="bicep_joint">
             <command_interface name="position">
@@ -38,8 +49,4 @@
             <state_interface name="position"/>
         </joint>
-        <joint name="rightClaw_joint">
-            <param name="mimic">leftClaw_joint</param>
-            <param name="multiplier">-1</param>
-        </joint>
     </ros2_control>
 </robot>
